File: Basic_Clock/_autosave-Basic_Clock.sch (KiCad schematic (older format))
At the start: 26 parts, among them J1 Conn_01x04_Female, J2 Conn_01x04_Female, J3 Conn_01x04_Female, SW1 SW_Push, SW2 SW_Push, SW3 SW_Push, SW4 SW_Push, U1 LM317_TO-220, U2 ATmega328P-PU, Y1 16Mhz

Commit message: Footprint somehow changed? Fixed and routed the missing with VIAs.
Parts:
- U2: footprint ATMEGA:DIP-28_W7.62mm_Socket -> Package_DIP:DIP-28_W7.62mm_Socket
Changed lines of the file:
@@
 F 0 "U2" H 2706 3846 50  0000 R CNN
 F 1 "ATmega328P-PU" H 2706 3755 50  0000 R CNN
-F 2 "ATMEGA:DIP-28_W7.62mm_Socket" H 3350 3800 50  0001 C CIN
+F 2 "Package_DIP:DIP-28_W7.62mm_Socket" H 3350 3800 50  0001 C CIN
 F 3 "https://www.distrelec.ch/Web/Downloads/_t/ds/ATMEGA328-AU_eng_tds.pdf" H 3350 3800 50  0001 C CNN
 	1    3350 3800
