File: Basic_Clock/Basic_Clock.kicad_pcb (KiCad board)
At the start: 2 copper layers, 97.8 x 71.1 mm, 26 parts, among them J1 Conn_01x04_Female, J2 Conn_01x04_Female, J3 Conn_01x04_Female, SW1 SW_Push, SW2 SW_Push, SW3 SW_Push, SW4 SW_Push, U1 LM317_TO-220, U2 ATmega328P-PU, Y1 16Mhz

Commit message: Footprint somehow changed? Fixed and routed the missing with VIAs.
Routing:
- net /RE: track 0.00 -> 68.1 mm, vias 0 -> 2
- net /DE: track 0.00 -> 54.5 mm, vias 0 -> 2
- net +5V: track 175.4 -> 185.1 mm, vias 0 -> 2

Commit message: Revisioned after Feedback from Frank.
Parts:
- added J-GND1: Conn_01x01_Male, Connector_Wire:SolderWirePad_1x01_Drill0.8mm, F.Cu at (52.1, 108.0)
- added J-VCC1: Conn_01x01_Male, Connector_Wire:SolderWirePad_1x01_Drill0.8mm, F.Cu at (47.0, 108.0)
- added R7: 10k, Resistor:R_Axial_DIN0411_L9.9mm_D3.6mm_P15.24mm_Horizontal, F.Cu at (88.9, 106.7)
- R4, R5, R6: value 1k -> 10k
- SW1: value SW_Push -> SW_Push_Reset
- moved SW4 44.5 mm to (62.2, 151.1), turned to 90 degrees
- moved SW3 39.4 mm to (72.4, 146.1), turned to 90 degrees
- moved SW2 34.5 mm to (82.5, 141.0), turned to 90 degrees
- moved R6 26.8 mm to (66.0, 106.7), turned to 270 degrees
- moved R5 26.7 mm to (73.7, 106.7), turned to 270 degrees
- moved R4 26.7 mm to (81.3, 106.7), turned to 270 degrees
- moved Y1 24.1 mm to (48.3, 156.2)
- moved C1 24.1 mm to (40.6, 148.6)
- moved C2 24.1 mm to (40.6, 167.6)
- moved SW1 15.2 mm to (120.7, 111.8)
- moved C5 6.35 mm to (59.7, 116.8)
Connections:
- R4 pad 1: /PIN2 -> +5V
- R4 pad 2: Net-(R4-Pad2) -> /PIN2
- R5 pad 1: /PIN3 -> +5V
- R5 pad 2: Net-(R5-Pad2) -> /PIN3
- R6 pad 1: /PIN4 -> +5V
- R6 pad 2: Net-(R6-Pad2) -> /PIN4
- SW2 pad 2: Net-(R4-Pad2) -> /PIN2
- SW3 pad 2: Net-(R5-Pad2) -> /PIN3
- SW4 pad 2: Net-(R6-Pad2) -> /PIN4
- U2 pad 15: /RE -> Net-(U2-Pad15)
- U2 pad 16: /DE -> Net-(U2-Pad16)
- U2 pad 25: Net-(U2-Pad25) -> /RE
- U2 pad 26: Net-(U2-Pad26) -> /DE
Routing:
- net GND: track 335.9 -> 12.4 mm
- net +5V: track 185.1 -> 30.7 mm
- net /RE: track 68.1 -> 34.1 mm, vias 2 -> 0
- net /DE: track 54.5 -> 25.4 mm, vias 2 -> 1
- net Net-(C2-Pad2): track 31.6 -> 55.7 mm
- net Net-(C1-Pad2): track 32.4 -> 56.5 mm
- net /PIN4: track 41.1 -> 61.1 mm
- net Net-(R7-Pad2): track 32.4 -> 49.1 mm
- net /PIN3: track 31.2 -> 46.9 mm
- net Net-(R4-Pad2): track 15.5 -> 0.00 mm
- net Net-(R6-Pad2): track 14.9 -> 0.00 mm
- net Net-(R5-Pad2): track 14.0 -> 0.00 mm
- net /PIN2: track 21.2 -> 34.0 mm
- net +28V: track 13.2 -> 20.1 mm
- net Net-(U2-Pad16): vias 0 -> 1
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- added copper zone on F.Cu, net +5V
- added copper zone on B.Cu, net GND
Other:
- board text added: "GND A B +5V"
- board text added: "SDA SCL GND +5V"
- board text added: "TX DE RE RX"
