File: PCBs/Basic_Clock_v0.5/Basic_Clock.kicad_pcb (KiCad board)
At the start: 2 copper layers, 97.8 x 71.1 mm, 34 parts, among them J1 Conn_01x04_Female, J3 Screw_Terminal_01x02, J4 Screw_Terminal_01x02, J5 Conn_01x03_Female, SW2 SW_Push, SW3 SW_Push, SW4 SW_Push, U1 LM317_TO-220, U2 ATmega328P-PU, U3 MAX485E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

Commit message: Update after Feedback.
Parts:
- added ICSP1: Conn_02x03_Odd_Even, Connector_PinSocket_2.54mm:PinSocket_2x03_P2.54mm_Vertical, F.Cu at (113.0, 168.9)
- added J_I2C2: Conn_01x02_Female, Connector THT:PinSocket_1x02_P2.54mm_Vertical, F.Cu at (94.0, 139.7)
- added U4: R-78E5.0-0.5, Converter_DCDC:Converter_DCDC_RECOM_R-78E-0.5_THT, F.Cu at (41.9, 149.9)
- moved J_POWER1 5.08 mm to (44.5, 165.1)
- moved R6 2.54 mm to (71.1, 109.2)
Connections:
- U2 pad 17: GND -> /MOSI
- U2 pad 18: GND -> /MISO
- U2 pad 19: GND -> /SCK
- U2 pad 2: GND -> /RXD
- U2 pad 3: GND -> /TXD
Routing:
- net Net-(ICSP1-Pad5): track 20.0 -> 82.6 mm
- net /MOSI: track 0.00 -> 25.9 mm
- net +28V: track 44.3 -> 61.4 mm
- net /SCK: track 0.00 -> 10.3 mm
- net /MISO: track 0.00 -> 10.3 mm
- net /TXD: track 0.00 -> 3.81 mm
- net /RXD: track 0.00 -> 3.81 mm
- net /PIN13: track 71.3 -> 73.8 mm
- net /RS485TX: track 27.3 -> 28.8 mm
- net Net-(R1-Pad2): track 24.0 -> 23.0 mm
- net /RS485RX: track 35.3 -> 36.0 mm
Other:
- board text added: "GND +28V"
- board text added: "GND +5V"
- board text added: "RX DE TX"
- board text added: "SCL SDA"
- board text added: "TX RX"
