File: PCBs/Basic_Clock_v0.5/Basic_Clock.sch (KiCad schematic (older format))
At the start: 34 parts, among them J1 Conn_01x04_Female, J3 Screw_Terminal_01x02, J4 Screw_Terminal_01x02, J5 Conn_01x03_Female, SW2 SW_Push, SW3 SW_Push, SW4 SW_Push, U1 LM317_TO-220, U2 ATmega328P-PU, U3 MAX485E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

Commit message: Update after Feedback.
Parts:
- added ICSP1: Conn_02x03_Odd_Even, Connector_PinSocket_2.54mm:PinSocket_2x03_P2.54mm_Vertical, symbol Connector_Generic:Conn_02x03_Odd_Even
- added J_I2C2: Conn_01x02_Female, Connector THT:PinSocket_1x02_P2.54mm_Vertical, symbol Connector:Conn_01x02_Female
- added U4: R-78E5.0-0.5, Converter_DCDC:Converter_DCDC_RECOM_R-78E-0.5_THT, symbol Regulator_Switching:R-78E5.0-0.5
Connections:
- net +28V: now also U4.1 (IN)
- net +5V: now also ICSP1.2 (Pin_2), U4.3 (OUT)
- net GND: now also ICSP1.6 (Pin_6), U4.2 (GND); no longer U2.17 (PB3), U2.18 (PB4), U2.19 (PB5), U2.2 (PD0), U2.3 (PD1)
- net at R7.2, U2.1 (~RESET~/PC6): now also ICSP1.5 (Pin_5)
- new net MISO: ICSP1.1 (Pin_1), U2.18 (PB4)
- new net MOSI: ICSP1.4 (Pin_4), U2.17 (PB3)
- new net RXD: J_I2C2.1 (Pin_1), U2.2 (PD0)
- new net SCK: ICSP1.3 (Pin_3), U2.19 (PB5)
- new net TXD: J_I2C2.2 (Pin_2), U2.3 (PD1)
Other:
- moved on the sheet: D1, J1, J5, R3
