File: PCBs/Basic_Clock_v1.0/Basic_Clock.kicad_pcb (KiCad board)
At the start: 2 copper layers, 80 x 71.1 mm, 28 parts, among them J1 Conn_01x04_Female, J2 Screw_Terminal_01x04, J3 Screw_Terminal_01x02, J4 Screw_Terminal_01x02, J5 Conn_01x03_Female, U2 ATmega328P-PU, U3 MAX485E, U4 R-78E5.0-0.5, Y1 16Mhz

Commit message: PCB latest version.
Parts:
- added J6: Screw_Terminal_01x02, TerminalBlock_RND:TerminalBlock_RND_205-00232_1x02_P5.08mm_Horizontal, F.Cu at (100.3, 109.2)
- moved J4 70.0 mm to (129.5, 114.8), turned to 270 degrees
- moved U4 64.1 mm to (119.4, 108.7), turned to 180 degrees
- moved R3 57.0 mm to (72.4, 160.3), turned to 90 degrees
- moved D1 55.5 mm to (72.4, 138.7), turned to 270 degrees
- moved J_POWER1 32.6 mm to (72.4, 130.0)
- moved J3 8.89 mm to (129.5, 128.3)
- moved R8 8.89 mm to (120.7, 124.5)
- moved H1 7.12 mm to (66.8, 108.2)
- moved H3 6.86 mm to (66.5, 170.4)
- moved J2 6.35 mm to (89.4, 170.2)
- moved J1 5.09 mm to (114.6, 141.0)
Routing:
- net /PIN11: track 84.7 -> 70.3 mm
- net Net-(J3-Pad2): track 18.8 -> 27.7 mm
- net +28V: track 26.0 -> 34.6 mm
- net /PIN13: track 66.1 -> 61.0 mm
- net /PIN12: track 72.5 -> 67.5 mm
- net /SDA: track 10.5 -> 14.9 mm
- net /SCL: track 10.5 -> 14.9 mm
- net Net-(J3-Pad1): track 18.8 -> 18.2 mm
Other:
- board size 80 x 71.1 mm -> 72.6 x 71.1 mm
- board text added: "10k"
- board text added: "120"
- board text added: "1k"
- board text added: "22pF"
- board text added: "U"
