File: PCBs/Basic_Clock_v1.0/Basic_Clock.sch (KiCad schematic (older format))
At the start: 28 parts, among them J1 Conn_01x04_Female, J2 Screw_Terminal_01x04, J3 Screw_Terminal_01x02, J4 Screw_Terminal_01x02, J5 Conn_01x03_Female, U2 ATmega328P-PU, U3 MAX485E, U4 R-78E5.0-0.5, Y1 16Mhz

Commit message: PCB latest version.
Parts:
- added J6: Screw_Terminal_01x02, TerminalBlock_RND:TerminalBlock_RND_205-00232_1x02_P5.08mm_Horizontal, symbol Connector:Screw_Terminal_01x02
Connections:
- net +28V: now also J6.2 (Pin_2)
- net GND: now also J6.1 (Pin_1)
Other:
- moved on the sheet: J4
Changed lines of the file:
@@
 L Connector:Screw_Terminal_01x02 J4
 U 1 1 5F6F79AD
-P 1705 5490
-F 0 "J4" H 1785 5482 50  0000 L CNN
-F 1 "Screw_Terminal_01x02" H 1785 5391 50  0000 L CNN
-F 2 "TerminalBlock_RND:TerminalBlock_RND_205-00232_1x02_P5.08mm_Horizontal" H 1705 5490 50  0001 C CNN
-F 3 "~" H 1705 5490 50  0001 C CNN
-	1    1705 5490
+P 1805 5590
+F 0 "J4" H 1885 5582 50  0000 L CNN
+F 1 "Screw_Terminal_01x02" H 1885 5491 50  0000 L CNN
+F 2 "TerminalBlock_RND:TerminalBlock_RND_205-00232_1x02_P5.08mm_Horizontal" H 1805 5590 50  0001 C CNN
+F 3 "~" H 1805 5590 50  0001 C CNN
+	1    1805 5590
 	-1   0    0    1
 $EndComp
@@
 L power:GND #PWR0120
 U 1 1 5F6F929F
-P 2025 5500
-F 0 "#PWR0120" H 2025 5250 50  0001 C CNN
-F 1 "GND" H 2030 5327 50  0000 C CNN
-F 2 "" H 2025 5500 50  0001 C CNN
-F 3 "" H 2025 5500 50  0001 C CNN
-	1    2025 5500
+P 2125 5600
+F 0 "#PWR0120" H 2125 5350 50  0001 C CNN
+F 1 "GND" H 2130 5427 50  0000 C CNN
+F 2 "" H 2125 5600 50  0001 C CNN
+F 3 "" H 2125 5600 50  0001 C CNN
+	1    2125 5600
 	1    0    0    -1
 $EndComp
@@
 L power:+28V #PWR0119
 U 1 1 5F94A5A7
-P 2030 5390
-F 0 "#PWR0119" H 2030 5240 50  0001 C CNN
-F 1 "+28V" H 2045 5563 50  0000 C CNN
-F 2 "" H 2280 5440 50  0001 C CNN
-F 3 "" H 2280 5440 50  0001 C CNN
-	1    2030 5390
+P 2130 5490
+F 0 "#PWR0119" H 2130 5340 50  0001 C CNN
+F 1 "+28V" H 2145 5663 50  0000 C CNN
+F 2 "" H 2380 5540 50  0001 C CNN
+F 3 "" H 2380 5540 50  0001 C CNN
+	1    2130 5490
 	1    0    0    -1
 $EndComp
@@
 	5350 6500 5270 6500
 Wire Wire Line
-	1905 5390 2030 5390
-Wire Wire Line
-	1905 5490 2025 5490
-Wire Wire Line
-	2025 5490 2025 5500
+	2005 5490 2130 5490
+Wire Wire Line
+	2005 5590 2125 5590
+Wire Wire Line
+	2125 5590 2125 5600
 $Comp
 L Connector:Conn_01x02_Female J_POWER1
@@
 	1    0    0    -1
 $EndComp
+$Comp
+L Connector:Screw_Terminal_01x02 J6
+U 1 1 5FBCB04E
+P 2705 6090
+F 0 "J6" H 2785 6082 50  0000 L CNN
+F 1 "Screw_Terminal_01x02" H 2785 5991 50  0000 L CNN
+F 2 "TerminalBlock_RND:TerminalBlock_RND_205-00232_1x02_P5.08mm_Horizontal" H 2705 6090 50  0001 C CNN
+F 3 "~" H 2705 6090 50  0001 C CNN
+	1    2705 6090
+	-1   0    0    1
+$EndComp
+$Comp
+L power:GND #PWR08
+U 1 1 5FBCB054
+P 3025 6100
+F 0 "#PWR08" H 3025 5850 50  0001 C CNN
+F 1 "GND" H 3030 5927 50  0000 C CNN
+F 2 "" H 3025 6100 50  0001 C CNN
+F 3 "" H 3025 6100 50  0001 C CNN
+	1    3025 6100
+	1    0    0    -1
+$EndComp
+$Comp
+L power:+28V #PWR09
+U 1 1 5FBCB05A
+P 3030 5990
+F 0 "#PWR09" H 3030 5840 50  0001 C CNN
+F 1 "+28V" H 3045 6163 50  0000 C CNN
+F 2 "" H 3280 6040 50  0001 C CNN
+F 3 "" H 3280 6040 50  0001 C CNN
+	1    3030 5990
+	1    0    0    -1
+$EndComp
+Wire Wire Line
+	2905 5990 3030 5990
+Wire Wire Line
+	2905 6090 3025 6090
+Wire Wire Line
+	3025 6090 3025 6100
 $EndSCHEMATC
